Commit message: Update simulated camera model

File: Assignment 3-B/assignment_3b/turtlebot3/turtlebot3/turtlebot3_description/urdf/turtlebot3_burger.urdf (robot description, URDF)
Before this commit: robot turtlebot3_burger, 10 links, 9 joints
Links:
- link camera_link: geometry collision box size=0.038 0.038 0.027
Joints:
- joint camera_joint: origin xyz=0.073 -0.011 0.084 rpy=0 0 0 -> xyz=0.055 0.0 0.102 rpy=0 0 0
- joint camera_rgb_joint: origin xyz=0.003 0.011 0.009 rpy=0 0 0 -> xyz=0.0 0.0 -0.002 rpy=0 0 0
